Commit message: Angle camera directly down

File: mini-project4/setup_files/hummingbird_base.xacro (robot description, xacro)
@@ -44,5 +44,5 @@
     enable_visual="true">
 	<box size="0.02 0.02 0.02" />
-	<origin xyz="0 0 ${arm_length/4}" rpy="0 ${-pi/6} 0" />
+	<origin xyz="0 0 ${-arm_length/3}" rpy="0 ${pi/2} 0" />
     </xacro:camera_macro>
   <xacro:if value="$(arg enable_ground_truth)">
